Commit message: removed inertia, added effort and velocity limits from indigo dev

File: schunk_description/urdf/lwa4d/lwa4d.gazebo.xacro (robot description, xacro)
@@ -2,35 +2,43 @@
 <robot xmlns:xacro="http://www.ros.org/wiki/xacro">
   <xacro:macro name="schunk_lwa4d_gazebo" params="name">
-    <gazebo reference="${name}_0_link">
-      <material value="Schunk/DarkGolden" />
-      <turnGravityOff>false</turnGravityOff>
+    <gazebo reference="${name}_base_link">
+      <gravity>true</gravity>
+      <self_collide>false</self_collide>
+      <material value="Schunk/Black"/>
     </gazebo>
     <gazebo reference="${name}_1_link">
-      <material value="Schunk/DarkGolden" />
-      <turnGravityOff>false</turnGravityOff>
+      <gravity>true</gravity>
+      <self_collide>false</self_collide>
+      <material value="Schunk/LightGrey"/>
     </gazebo>
     <gazebo reference="${name}_2_link">
-      <material value="Schunk/DarkGolden" />
-      <turnGravityOff>false</turnGravityOff>
+      <gravity>true</gravity>
+      <self_collide>false</self_collide>
+      <material value="Schunk/Black"/>
     </gazebo>
     <gazebo reference="${name}_3_link">
-      <material value="Schunk/DarkGolden" />
-      <turnGravityOff>false</turnGravityOff>
+      <gravity>true</gravity>
+      <self_collide>false</self_collide>
+      <material value="Schunk/LightGrey"/>
     </gazebo>
     <gazebo reference="${name}_4_link">
-      <material value="Schunk/DarkGolden" />
-      <turnGravityOff>false</turnGravityOff>
+      <gravity>true</gravity>
+      <self_collide>false</self_collide>
+      <material value="Schunk/Black"/>
     </gazebo>
     <gazebo reference="${name}_5_link">
-      <material value="Schunk/DarkGolden" />
-      <turnGravityOff>false</turnGravityOff>
+      <gravity>true</gravity>
+      <self_collide>false</self_collide>
+      <material value="Schunk/LightGrey"/>
     </gazebo>
     <gazebo reference="${name}_6_link">
-      <material value="Schunk/DarkGolden" />
-      <turnGravityOff>false</turnGravityOff>
+      <gravity>true</gravity>
+      <self_collide>false</self_collide>
+      <material value="Schunk/Black"/>
     </gazebo>
     <gazebo reference="${name}_7_link">
-      <material value="Schunk/DarkGolden" />
-      <turnGravityOff>false</turnGravityOff>
+      <gravity>true</gravity>
+      <self_collide>false</self_collide>
+      <material value="Schunk/LightGrey"/>
     </gazebo>
   </xacro:macro>

File: schunk_description/urdf/lwa4d/lwa4d.urdf.xacro (robot description, xacro)
@@ -11,9 +11,10 @@
     </joint>
     <link name="${name}_0_link">
-      <inertial>
+      <xacro:default_inertial/>
+      <!--inertial>
         <origin xyz="0 0 0" rpy="0 0 0"/>
         <mass value="1.0"/>
         <inertia ixx="0.01" ixy="0" ixz="0" iyy="0.01" iyz="0" izz="0.01" />
-      </inertial>
+      </inertial-->
       <visual>
         <origin xyz="0 0 0.004" rpy="0 0 0" />
@@ -38,14 +39,15 @@
       <calibration rising="${arm_1_ref}"/>
       <dynamics damping="10" />
-      <limit effort="370" velocity="2.0" lower="-3.1" upper="3.1"/>
+      <limit effort="216" velocity="0.43633" lower="-3.1" upper="3.1"/>
       <safety_controller k_position="20" k_velocity="50" soft_lower_limit="${-3.1 + 0.01}" soft_upper_limit="${3.1 - 0.01}" />
     </joint>
     <link name="${name}_1_link">
-      <inertial>
+      <xacro:default_inertial/>
+      <!--inertial>
         <origin xyz="0 0 0" rpy="0 0 0" />
         <!--mass value="5.9907"/-->
-        <mass value="2.0"/>
-        <inertia ixx="0.01" ixy="0" ixz="0" iyy="0.01" iyz="0" izz="0.01" />
-      </inertial>
+        <!--mass value="2.0"/>
+        <inertia ixx="0.01" ixy="0" ixz="0" iyy="0.01" iyz="0" izz="0.01" />
+      </inertial-->
       <visual>
         <origin xyz="0 0 -0.15" rpy="0 0 ${M_PI}" />
@@ -70,13 +72,14 @@
       <calibration rising="${arm_2_ref}"/>
       <dynamics damping="10" />
-      <limit effort="370" velocity="2.0" lower="-2.14675498" upper="2.14675498"/>
-      <safety_controller k_position="20" k_velocity="50" soft_lower_limit="${-2.14675498 + 0.01}"   soft_upper_limit="${2.14675498 - 0.01}" />
+      <limit effort="216" velocity="0.43633" lower="-2.14" upper="2.14"/>
+      <safety_controller k_position="20" k_velocity="50" soft_lower_limit="${-2.14 + 0.01}"   soft_upper_limit="${2.14 - 0.01}" />
     </joint>
     <link name="${name}_2_link">
-      <inertial>
+      <xacro:default_inertial/>
+      <!--inertial>
         <origin xyz="0 0 0" rpy="0 0 0"/>
         <mass value="2.0"/>
         <inertia ixx="0.03" ixy="0" ixz="0" iyy="0.03" iyz="0" izz="0.03" />
-      </inertial>
+      </inertial-->
       <visual>
         <origin xyz="0 0 0" rpy="0 0 ${M_PI}" />
@@ -101,13 +104,14 @@
       <calibration rising="${arm_3_ref}"/>
       <dynamics damping="5" />
-      <limit effort="176" velocity="2.0" lower="-3.141592654" upper="3.141592654"/>
-      <safety_controller k_position="20" k_velocity="25" soft_lower_limit="${-3.141592654 + 0.01}" soft_upper_limit="${3.141592654 - 0.01}" />
+      <limit effort="81.5" velocity="0.4189" lower="-M_PI" upper="M_PI"/>
+      <safety_controller k_position="20" k_velocity="25" soft_lower_limit="${-M_PI + 0.01}" soft_upper_limit="${M_PI - 0.01}" />
     </joint>
     <link name="${name}_3_link">
-      <inertial>
+      <xacro:default_inertial/>
+      <!--inertial>
         <origin xyz="0 0 0" rpy="0 0 0"/>
         <mass value="2.0"/>
         <inertia ixx="0.03" ixy="0" ixz="0" iyy="0.03" iyz="0" izz="0.03" />
-      </inertial>
+      </inertial-->
       <visual>
         <origin xyz="0 0 -0.328" rpy="0 0 ${M_PI}" />
@@ -132,13 +136,14 @@
       <calibration rising="${arm_4_ref}"/>
       <dynamics damping="5" />
-      <limit effort="176" velocity="2.0" lower="-2.181661565" upper="2.181661565"/>
-      <safety_controller k_position="20" k_velocity="25" soft_lower_limit="${-2.181661565 + 0.01}" soft_upper_limit="${2.181661565 - 0.01}" />
+      <limit effort="176" velocity="2.0" lower="-2.18" upper="2.18"/>
+      <safety_controller k_position="20" k_velocity="25" soft_lower_limit="${-2.18 + 0.01}" soft_upper_limit="${2.18 - 0.01}" />
     </joint>
     <link name="${name}_4_link">
-      <inertial>
+      <xacro:default_inertial/>
+      <!--inertial>
         <origin xyz="0 0 0" rpy="0 0 0"/>
         <mass value="2.0"/>
         <inertia ixx="0.03" ixy="0" ixz="0" iyy="0.03" iyz="0" izz="0.03" />
-      </inertial>
+      </inertial-->
       <visual>
         <origin xyz="0 0 0" rpy="0 0 ${M_PI}" />
@@ -163,13 +168,14 @@
       <calibration rising="${arm_5_ref}"/>
       <dynamics damping="5" />
-      <limit effort="41.6" velocity="2.0" lower="-3.141592654" upper="3.141592654" />
-      <safety_controller k_position="20" k_velocity="25" soft_lower_limit="${-3.141592654 + 0.01}" soft_upper_limit="${3.141592654 - 0.01}" />
+      <limit effort="20.7" velocity="0.43633" lower="-M_PI" upper="M_PI" />
+      <safety_controller k_position="20" k_velocity="25" soft_lower_limit="${-M_PI + 0.01}" soft_upper_limit="${M_PI - 0.01}" />
     </joint>
     <link name="${name}_5_link">
-      <inertial>
+      <xacro:default_inertial/>
+      <!--inertial>
         <origin xyz="0 0 0" rpy="0 0 0"/>
         <mass value="2.313272"/>
         <inertia ixx="0.03" ixy="0" ixz="0" iyy="0.03" iyz="0" izz="0.03" />
-      </inertial>
+      </inertial-->
       <visual>
         <origin xyz="0 0 -0.323" rpy="0 0 ${M_PI}" />
@@ -194,13 +200,14 @@
       <calibration rising="${arm_6_ref}"/>
       <dynamics damping="5" />
-      <limit effort="20.1" velocity="2.0" lower="-2.0" upper="2.0" />
-      <safety_controller k_position="20" k_velocity="25" soft_lower_limit="${-2.967059728 + 0.01}" soft_upper_limit="${2.967059728 - 0.01}" />
+      <limit effort="15" velocity="1.2566" lower="-2.0" upper="2.0" />
+      <safety_controller k_position="20" k_velocity="25" soft_lower_limit="${-2.0 + 0.01}" soft_upper_limit="${2.0 - 0.01}" />
     </joint>
     <link name="${name}_6_link">
-      <inertial>
+      <xacro:default_inertial/>
+      <!--inertial>
         <origin xyz="0 0 0" rpy="0 0 0"/>
         <mass value="2.057856"/>
         <inertia ixx="0.01" ixy="0" ixz="0" iyy="0.01" iyz="0" izz="0.01" />
-      </inertial>
+      </inertial-->
       <visual>
         <origin xyz="0 0 0" rpy="0 ${M_PI} 0" />
@@ -225,13 +232,14 @@
       <calibration rising="${arm_7_ref}"/>
       <dynamics damping="5" />
-      <limit effort="9.6" velocity="2.0" lower="-2.967059728" upper="2.967059728" />
+      <limit effort="15" velocity="1.2566" lower="-2.967059728" upper="2.967059728" />
       <safety_controller k_position="20" k_velocity="25" soft_lower_limit="${-2.967059728 + 0.01}" soft_upper_limit="${2.967059728 - 0.01}" />
     </joint>
     <link name="${name}_7_link">
-      <inertial>
+      <xacro:default_inertial/>
+      <!--inertial>
         <origin xyz="0 0 0" rpy="0 0 0"/>
         <mass value="1.120198"/>
         <inertia ixx="0.01" ixy="0" ixz="0" iyy="0.01" iyz="0" izz="0.01" />
-      </inertial>
+      </inertial-->
       <visual>
         <origin xyz="0 0 0" rpy="0 0 0" />
