Commit message: joint_limits corrected and added finger for pg70

File: schunk_description/urdf/lwa4d/lwa4d.urdf.xacro (robot description, xacro)
@@ -38,6 +38,6 @@
       <calibration rising="${arm_1_ref}"/>
       <dynamics damping="10" />
-      <limit effort="370" velocity="2.0" lower="-6.2831853" upper="6.2831853"/>
-      <safety_controller k_position="20" k_velocity="50" soft_lower_limit="${-6.2831853 + 0.01}" soft_upper_limit="${6.2831853 - 0.01}" />
+      <limit effort="370" velocity="2.0" lower="-3.438" upper="2.846"/>
+      <safety_controller k_position="20" k_velocity="50" soft_lower_limit="${-3.438 + 0.01}" soft_upper_limit="${2.846 - 0.01}" />
     </joint>
     <link name="${name}_1_link">
@@ -70,6 +70,6 @@
       <calibration rising="${arm_2_ref}"/>
       <dynamics damping="10" />
-      <limit effort="370" velocity="2.0" lower="-1.97" upper="1.97"/>
-      <safety_controller k_position="20" k_velocity="50" soft_lower_limit="${-1.97 + 0.01}"   soft_upper_limit="${1.97 - 0.01}" />
+      <limit effort="370" velocity="2.0" lower="-2.14675498" upper="2.14675498"/>
+      <safety_controller k_position="20" k_velocity="50" soft_lower_limit="${-2.14675498 + 0.01}"   soft_upper_limit="${2.14675498 - 0.01}" />
     </joint>
     <link name="${name}_2_link">
@@ -101,6 +101,6 @@
       <calibration rising="${arm_3_ref}"/>
       <dynamics damping="5" />
-      <limit effort="176" velocity="2.0" lower="-6.2831853" upper="6.2831853"/>
-      <safety_controller k_position="20" k_velocity="25" soft_lower_limit="${-6.2831853 + 0.01}" soft_upper_limit="${6.2831853 - 0.01}" />
+      <limit effort="176" velocity="2.0" lower="-3.141592654" upper="3.141592654"/>
+      <safety_controller k_position="20" k_velocity="25" soft_lower_limit="${-3.141592654 + 0.01}" soft_upper_limit="${3.141592654 - 0.01}" />
     </joint>
     <link name="${name}_3_link">
@@ -132,6 +132,6 @@
       <calibration rising="${arm_4_ref}"/>
       <dynamics damping="5" />
-      <limit effort="176" velocity="2.0" lower="-2.08208" upper="2.08208"/>
-      <safety_controller k_position="20" k_velocity="25" soft_lower_limit="${-2.08208 + 0.01}" soft_upper_limit="${2.08208 - 0.01}" />
+      <limit effort="176" velocity="2.0" lower="-2.181661565" upper="2.181661565"/>
+      <safety_controller k_position="20" k_velocity="25" soft_lower_limit="${-2.181661565 + 0.01}" soft_upper_limit="${2.181661565 - 0.01}" />
     </joint>
     <link name="${name}_4_link">
@@ -163,6 +163,6 @@
       <calibration rising="${arm_5_ref}"/>
       <dynamics damping="5" />
-      <limit effort="41.6" velocity="2.0" lower="-6.2831853" upper="6.2831853" />
-      <safety_controller k_position="20" k_velocity="25" soft_lower_limit="${-6.2831853 + 0.01}" soft_upper_limit="${6.2831853 - 0.01}" />
+      <limit effort="41.6" velocity="2.0" lower="-3.141592654" upper="3.141592654" />
+      <safety_controller k_position="20" k_velocity="25" soft_lower_limit="${-3.141592654 + 0.01}" soft_upper_limit="${3.141592654 - 0.01}" />
     </joint>
     <link name="${name}_5_link">
@@ -194,6 +194,6 @@
       <calibration rising="${arm_6_ref}"/>
       <dynamics damping="5" />
-      <limit effort="20.1" velocity="2.0" lower="-1.8" upper="1.8" />
-      <safety_controller k_position="20" k_velocity="25" soft_lower_limit="${-1.8 + 0.01}" soft_upper_limit="${1.8 - 0.01}" />
+      <limit effort="20.1" velocity="2.0" lower="-2.0" upper="2.0" />
+      <safety_controller k_position="20" k_velocity="25" soft_lower_limit="${-2.967059728 + 0.01}" soft_upper_limit="${2.967059728 - 0.01}" />
     </joint>
     <link name="${name}_6_link">
@@ -225,6 +225,6 @@
       <calibration rising="${arm_7_ref}"/>
       <dynamics damping="5" />
-      <limit effort="9.6" velocity="2.0" lower="-6.2831853" upper="6.2831853" />
-      <safety_controller k_position="20" k_velocity="25" soft_lower_limit="${-6.2831853 + 0.01}" soft_upper_limit="${6.2831853 - 0.01}" />
+      <limit effort="9.6" velocity="2.0" lower="-2.967059728" upper="2.967059728" />
+      <safety_controller k_position="20" k_velocity="25" soft_lower_limit="${-2.967059728 + 0.01}" soft_upper_limit="${2.967059728 - 0.01}" />
     </joint>
     <link name="${name}_7_link">

File: schunk_description/urdf/pg70/pg70.urdf.xacro (robot description, xacro)
@@ -35,7 +35,7 @@
       <parent link="${name}_gripper_link" />
       <child link="${name}_finger_left_link" />
-      <limit effort="100" lower="-0.001" upper="0.0345" velocity="2.0"/>
+      <limit effort="100" lower="-0.001" upper="0.033" velocity="2.0"/>
       <calibration rising="${pg70_finger_left_ref}"/>
-      <origin xyz="0 0.0105 0.0789" rpy="0 0 0"/>
+      <origin xyz="0 0.0105 ${0.0789-0.01}" rpy="0 0 0"/>
       <axis xyz="0 1 0" />
     </joint>
@@ -47,6 +47,7 @@
       </inertial>
       <visual>
+        <origin xyz="0 0 0.05" rpy="0 0 0" />
         <geometry>
-          <box size="0.03 0.01 0.01"/>
+          <box size="0.03 0.02 0.10"/>
         </geometry>
         <material name="black">
@@ -55,6 +56,7 @@
       </visual>
       <collision>
+        <origin xyz="0 0 0.05" rpy="0 0 0" />
         <geometry>
-          <box size="0.03 0.01 0.01"/>
+          <box size="0.03 0.02 0.10"/>
         </geometry>
         <material name="black">
@@ -67,7 +69,7 @@
       <parent link="${name}_gripper_link" />
       <child link="${name}_finger_right_link" />
-      <limit effort="100" lower="-0.001" upper="0.0345" velocity="2.0"/>
+      <limit effort="100" lower="-0.001" upper="0.033" velocity="2.0"/>
       <calibration rising="${pg70_finger_right_ref}"/>
-      <origin xyz="0 -0.0105 0.0789" rpy="-0 0 0"/>
+      <origin xyz="0 -0.0105 ${0.0789-0.01}" rpy="-0 0 0"/>
       <axis xyz="0 -1 0" />
     </joint>
@@ -79,6 +81,7 @@
       </inertial>
       <visual>
+        <origin xyz="0 0 0.05" rpy="0 0 0" />
         <geometry>
-          <box size="0.03 0.01 0.01"/>
+          <box size="0.03 0.02 0.10"/>
         </geometry>
         <material name="black">
@@ -87,6 +90,7 @@
       </visual>
       <collision>
+        <origin xyz="0 0 0.05" rpy="0 0 0" />
         <geometry>
-          <box size="0.03 0.01 0.01"/>
+          <box size="0.03 0.02 0.10"/>
         </geometry>
         <material name="black">

Commit message: joint limit changed

File: schunk_description/urdf/lwa4d/lwa4d.urdf.xacro (robot description, xacro)
@@ -32,5 +32,5 @@
     <!-- joint between arm_0_link and arm_1_link -->
     <joint name="${name}_1_joint" type="revolute">
-      <origin xyz="0 0 0.15" rpy="0 -${M_PI} 0"/>
+      <origin xyz="0 0 0.15" rpy="0 -${M_PI} ${M_PI}"/>
       <parent link="${name}_0_link"/>
       <child link="${name}_1_link"/>
@@ -38,6 +38,6 @@
       <calibration rising="${arm_1_ref}"/>
       <dynamics damping="10" />
-      <limit effort="370" velocity="2.0" lower="-3.438" upper="2.846"/>
-      <safety_controller k_position="20" k_velocity="50" soft_lower_limit="${-3.438 + 0.01}" soft_upper_limit="${2.846 - 0.01}" />
+      <limit effort="370" velocity="2.0" lower="-3.1" upper="3.1"/>
+      <safety_controller k_position="20" k_velocity="50" soft_lower_limit="${-3.1 + 0.01}" soft_upper_limit="${3.1 - 0.01}" />
     </joint>
     <link name="${name}_1_link">

Commit message: urdf fixed

File: schunk_description/urdf/lwa4d/lwa4d.urdf.xacro (robot description, xacro)
@@ -45,5 +45,5 @@
       <xacro:default_inertial/>
       <!--inertial>
-        <origin xyz="0 0 0" rpy="0 0 0" />
+        <origin xyz="0 0 0" rpy="0 0 0" /-->
         <!--mass value="5.9907"/-->
         <!--mass value="2.0"/>
@@ -104,5 +104,5 @@
       <calibration rising="${arm_3_ref}"/>
       <dynamics damping="5" />
-      <limit effort="81.5" velocity="0.4189" lower="-M_PI" upper="M_PI"/>
+      <limit effort="81.5" velocity="0.4189" lower="${-M_PI}" upper="${M_PI}"/>
       <safety_controller k_position="20" k_velocity="25" soft_lower_limit="${-M_PI + 0.01}" soft_upper_limit="${M_PI - 0.01}" />
     </joint>
@@ -168,5 +168,5 @@
       <calibration rising="${arm_5_ref}"/>
       <dynamics damping="5" />
-      <limit effort="20.7" velocity="0.43633" lower="-M_PI" upper="M_PI" />
+      <limit effort="20.7" velocity="0.43633" lower="${-M_PI}" upper="${M_PI}" />
       <safety_controller k_position="20" k_velocity="25" soft_lower_limit="${-M_PI + 0.01}" soft_upper_limit="${M_PI - 0.01}" />
     </joint>
