Commit message: alte version von lwa4d

File: schunk_description/urdf/lwa4d/lwa4d.urdf.xacro (robot description, xacro)
@@ -1,74 +1,64 @@
 <?xml version="1.0"?>
 <robot xmlns:xacro="http://www.ros.org/wiki/xacro">
-  <property name="safety_offset" value="0.01"/>
-  <xacro:include filename="$(find schunk_description)/urdf/lwa4d/lwa4d.gazebo.xacro"/>
-  <xacro:include filename="$(find schunk_description)/urdf/lwa4d/lwa4d.transmission.xacro"/>
-  <xacro:macro name="schunk_lwa4d" params="parent name *origin arm_1_ref arm_2_ref arm_3_ref arm_4_ref arm_5_ref arm_6_ref arm_7_ref has_podest">
-    <xacro:if value="${has_podest}">
-      <!-- joint between base_link and lwa4p_extended_connector_link -->
-      <joint name="${name}_podest_joint" type="fixed">
-        <insert_block name="origin" />
-        <parent link="${parent}"/>
-        <child link="${name}_podest_link"/>
-      </joint>
-      <link name="${name}_podest_link">
-        <xacro:default_inertial/>
-        <visual>
-          <origin xyz="0 0 0" rpy="0 0 0" />
-          <geometry>
-            <cylinder radius="0.03" length="0.05"/>
-          </geometry>
-        </visual>
-        <collision>
-          <origin xyz="0 0 0" rpy="0 0 0" />
-          <geometry>
-            <cylinder radius="0.03" length="0.05"/>
-          </geometry>
-        </collision>
-      </link>
-      <joint name="${name}_base_joint" type="fixed">
-        <origin xyz="0 0 0.175" rpy="0 ${M_PI} 0" />
-        <parent link="${name}_podest_link"/>
-        <child link="${name}_base_link"/>
-      </joint>
-    </xacro:if>
-    <xacro:unless value="${has_podest}">
-      <!-- joint between base_link and lwa4p_extended_connector_link -->
-      <joint name="${name}_base_joint" type="fixed">
-        <insert_block name="origin" />
-        <parent link="${parent}"/>
-        <child link="${name}_base_link"/>
-      </joint>
-    </xacro:unless>
-    <link name="${name}_base_link">
-      <xacro:default_inertial/>
-    </link>
-    <!-- joint between arm_base_link and arm_1_link -->
+  <xacro:include filename="$(find schunk_description)/urdf/lwa4d/lwa4d.gazebo.xacro" />
+  <xacro:include filename="$(find schunk_description)/urdf/lwa4d/lwa4d.transmission.xacro" />
+  <xacro:macro name="schunk_lwa4d" params="parent name *origin">
+    <!-- joint between base_link and arm_0_link -->
+    <joint name="${name}_0_joint" type="fixed" >
+      <insert_block name="origin" />
+      <parent link="${parent}" />
+      <child link="${name}_0_link" />
+    </joint>
+    <link name="${name}_0_link">
+      <xacro:default_inertial/>
+      <!--inertial>
+        <origin xyz="0 0 0" rpy="0 0 0"/>
+        <mass value="1.0"/>
+        <inertia ixx="0.01" ixy="0" ixz="0" iyy="0.01" iyz="0" izz="0.01" />
+      </inertial-->
+      <visual>
+        <origin xyz="0 0 0.004" rpy="0 0 0" />
+        <geometry>
+          <cylinder radius="0.045" length="0.08"/>
+        </geometry>
+        <material name="Schunk/Black" />
+      </visual>
+      <collision>
+        <origin xyz="0 0 0.005" rpy="0 0 0" />
+        <geometry>
+          <box size="0.01 0.01 0.01"/>
+        </geometry>
+      </collision>
+    </link>
+    <!-- joint between arm_0_link and arm_1_link -->
     <joint name="${name}_1_joint" type="revolute">
-      <origin xyz="0 0 0" rpy="0 0 0" />
-      <parent link="${name}_base_link"/>
+      <origin xyz="0 0 0.15" rpy="0 -${M_PI} ${M_PI}"/>
+      <parent link="${name}_0_link"/>
       <child link="${name}_1_link"/>
       <axis xyz="0 0 1"/>
       <calibration rising="${arm_1_ref}"/>
-      <limit effort="216" velocity="0.43633" lower="${-M_PI+safety_offset}" upper="${M_PI-safety_offset}"/>
+      <dynamics damping="10" />
+      <limit effort="216" velocity="0.43633" lower="-3.1" upper="3.1"/>
+      <safety_controller k_position="20" k_velocity="50" soft_lower_limit="${-3.1 + 0.01}" soft_upper_limit="${3.1 - 0.01}" />
     </joint>
     <link name="${name}_1_link">
       <xacro:default_inertial/>
-<!--
-      <xacro:cylinder_inertial radius="0.06" length="0.150" mass="3.6">
-          <origin xyz="0 0 0.02" rpy="0 0 0"/>
-      </xacro:cylinder_inertial>
--->
-      <visual>
-        <origin xyz="0 0 -0.15" rpy="0 0 ${M_PI}"/>
-        <geometry>
-          <mesh filename="package://schunk_description/meshes/lwa4d/arm_1_link.stl"/>
-        </geometry>
-        <material name="Schunk/LightGrey"/>
-      </visual>
-      <collision>
-        <origin xyz="0 0 -0.15" rpy="0 0 ${M_PI}"/>
-        <geometry>
-          <mesh filename="package://schunk_description/meshes/lwa4d/arm_1_link.stl"/>
+      <!--inertial>
+        <origin xyz="0 0 0" rpy="0 0 0" /-->
+        <!--mass value="5.9907"/-->
+        <!--mass value="2.0"/>
+        <inertia ixx="0.01" ixy="0" ixz="0" iyy="0.01" iyz="0" izz="0.01" />
+      </inertial-->
+      <visual>
+        <origin xyz="0 0 -0.15" rpy="0 0 ${M_PI}" />
+        <geometry>
+          <mesh filename="package://schunk_description/meshes/lwa4d/arm_1_link.stl" />
+        </geometry>
+        <material name="Schunk/LightGrey" />
+      </visual>
+      <collision>
+        <origin xyz="0 0 -0.15" rpy="0 0 ${M_PI}" />
+        <geometry>
+          <mesh filename="package://schunk_description/meshes/lwa4d/arm_1_link.stl" />
         </geometry>
       </collision>
@@ -81,24 +71,26 @@
       <axis xyz="0 0 1"/>
       <calibration rising="${arm_2_ref}"/>
-      <limit effort="216" velocity="0.43633" lower="${-2.14 + safety_offset}" upper="${2.14 - safety_offset}"/>
+      <dynamics damping="10" />
+      <limit effort="216" velocity="0.43633" lower="-2.14" upper="2.14"/>
+      <safety_controller k_position="20" k_velocity="50" soft_lower_limit="${-2.14 + 0.01}"   soft_upper_limit="${2.14 - 0.01}" />
     </joint>
     <link name="${name}_2_link">
       <xacro:default_inertial/>
-<!--
-      <xacro:cylinder_inertial radius="0.06" length="0.150" mass="2.0">
-        <origin xyz="0 0 0" rpy="0 0 0"/>
-      </xacro:cylinder_inertial>
--->
-      <visual>
-        <origin xyz="0 0 0" rpy="0 0 ${M_PI}"/>
-        <geometry>
-          <mesh filename="package://schunk_description/meshes/lwa4d/arm_2_link.stl"/>
-        </geometry>
-        <material name="Schunk/Black"/>
-      </visual>
-      <collision>
-        <origin xyz="0 0 0" rpy="0 0 ${M_PI}"/>
-        <geometry>
-          <mesh filename="package://schunk_description/meshes/lwa4d/arm_2_link_collision.stl"/>
+      <!--inertial>
+        <origin xyz="0 0 0" rpy="0 0 0"/>
+        <mass value="2.0"/>
+        <inertia ixx="0.03" ixy="0" ixz="0" iyy="0.03" iyz="0" izz="0.03" />
+      </inertial-->
+      <visual>
+        <origin xyz="0 0 0" rpy="0 0 ${M_PI}" />
+        <geometry>
+          <mesh filename="package://schunk_description/meshes/lwa4d/arm_2_link.stl" />
+        </geometry>
+        <material name="Schunk/Black" />
+      </visual>
+      <collision>
+        <origin xyz="0 0 0" rpy="0 0 ${M_PI}" />
+        <geometry>
+          <mesh filename="package://schunk_description/meshes/lwa4d/arm_2_link.stl" />
         </geometry>
       </collision>
@@ -111,24 +103,26 @@
       <axis xyz="0 0 1"/>
       <calibration rising="${arm_3_ref}"/>
-      <limit effort="81.5" velocity="0.4189" lower="${-M_PI + safety_offset}" upper="${M_PI - safety_offset}"/>
+      <dynamics damping="5" />
+      <limit effort="81.5" velocity="0.4189" lower="${-M_PI}" upper="${M_PI}"/>
+      <safety_controller k_position="20" k_velocity="25" soft_lower_limit="${-M_PI + 0.01}" soft_upper_limit="${M_PI - 0.01}" />
     </joint>
     <link name="${name}_3_link">
       <xacro:default_inertial/>
-<!--
-      <xacro:cylinder_inertial radius="0.06" length="0.2" mass="2.0">
-        <origin xyz="0.0 0 -0.2" rpy="0 0 0"/>
-      </xacro:cylinder_inertial>
--->
-      <visual>
-        <origin xyz="0 0 -0.39" rpy="0 0 ${M_PI}"/>
-        <geometry>
-          <mesh filename="package://schunk_description/meshes/lwa4d/arm_3_link.stl"/>
-        </geometry>
-        <material name="Schunk/LightGrey"/>
-      </visual>
-      <collision>
-        <origin xyz="0 0 -0.39" rpy="0 0 ${M_PI}"/>
-        <geometry>
-          <mesh filename="package://schunk_description/meshes/lwa4d/arm_3_link_collision.stl"/>
+      <!--inertial>
+        <origin xyz="0 0 0" rpy="0 0 0"/>
+        <mass value="2.0"/>
+        <inertia ixx="0.03" ixy="0" ixz="0" iyy="0.03" iyz="0" izz="0.03" />
+      </inertial-->
+      <visual>
+        <origin xyz="0 0 -0.328" rpy="0 0 ${M_PI}" />
+        <geometry>
+          <mesh filename="package://schunk_description/meshes/lwa4d/arm_3_link.stl" />
+        </geometry>
+        <material name="Schunk/LightGrey" />
+      </visual>
+      <collision>
+        <origin xyz="0 0 -0.328" rpy="0 0 ${M_PI}" />
+        <geometry>
+          <mesh filename="package://schunk_description/meshes/lwa4d/arm_3_link.stl" />
         </geometry>
       </collision>
@@ -136,29 +130,31 @@
     <!-- joint between arm_3_link and arm_4_link -->
     <joint name="${name}_4_joint" type="revolute">
-      <origin xyz="0 0 -0.39" rpy="-${M_PI/2} 0 0"/>
+      <origin xyz="0 0 -0.328" rpy="-${M_PI/2} 0 0"/>
       <parent link="${name}_3_link"/>
       <child link="${name}_4_link"/>
-      <axis xyz="0 0 1"/>
+      <axis xyz="0 0 1" />
       <calibration rising="${arm_4_ref}"/>
-      <limit effort="81.5" velocity="0.4189" lower="${-2.18 + safety_offset}" upper="${2.18 - safety_offset}"/>
+      <dynamics damping="5" />
+      <limit effort="176" velocity="2.0" lower="-2.18" upper="2.18"/>
+      <safety_controller k_position="20" k_velocity="25" soft_lower_limit="${-2.18 + 0.01}" soft_upper_limit="${2.18 - 0.01}" />
     </joint>
     <link name="${name}_4_link">
       <xacro:default_inertial/>
-<!--
-      <xacro:cylinder_inertial radius="0.06" length="0.150" mass="1.2">
-        <origin xyz="0 0 0" rpy="0 0 0"/>
-      </xacro:cylinder_inertial>
--->
-      <visual>
-        <origin xyz="0 0 0" rpy="0 0 ${M_PI}"/>
-        <geometry>
-          <mesh filename="package://schunk_description/meshes/lwa4d/arm_4_link.stl"/>
-        </geometry>
-        <material name="Schunk/Black"/>
-      </visual>
-      <collision>
-        <origin xyz="0 0 0" rpy="0 0 ${M_PI}"/>
-        <geometry>
-          <mesh filename="package://schunk_description/meshes/lwa4d/arm_4_link_collision.stl"/>
+      <!--inertial>
+        <origin xyz="0 0 0" rpy="0 0 0"/>
+        <mass value="2.0"/>
+        <inertia ixx="0.03" ixy="0" ixz="0" iyy="0.03" iyz="0" izz="0.03" />
+      </inertial-->
+      <visual>
+        <origin xyz="0 0 0" rpy="0 0 ${M_PI}" />
+        <geometry>
+          <mesh filename="package://schunk_description/meshes/lwa4d/arm_4_link.stl" />
+        </geometry>
+        <material name="Schunk/Black" />
+      </visual>
+      <collision>
+        <origin xyz="0 0 0" rpy="0 0 ${M_PI}" />
+        <geometry>
+          <mesh filename="package://schunk_description/meshes/lwa4d/arm_4_link.stl" />
         </geometry>
       </collision>
@@ -166,29 +162,31 @@
     <!-- joint between arm_4_link and arm_5_link -->
     <joint name="${name}_5_joint" type="revolute">
-      <origin xyz="0 0 0" rpy="${M_PI/2} 0 0"/>
+      <origin xyz="0 0 0" rpy="${M_PI/2} 0 0" />
       <parent link="${name}_4_link"/>
       <child link="${name}_5_link"/>
-      <axis xyz="0 0 1"/>
+      <axis xyz="0 0 1" />
       <calibration rising="${arm_5_ref}"/>
-      <limit effort="20.7" velocity="0.43633" lower="${-M_PI + safety_offset}" upper="${M_PI - safety_offset}"/>
+      <dynamics damping="5" />
+      <limit effort="20.7" velocity="0.43633" lower="${-M_PI}" upper="${M_PI}" />
+      <safety_controller k_position="20" k_velocity="25" soft_lower_limit="${-M_PI + 0.01}" soft_upper_limit="${M_PI - 0.01}" />
     </joint>
     <link name="${name}_5_link">
       <xacro:default_inertial/>
-<!--
-      <xacro:cylinder_inertial radius="0.06" length="0.15" mass="1.2">
-        <origin xyz="0 0 -0.18" rpy="0 0 0"/>
-      </xacro:cylinder_inertial>
--->
-      <visual>
-        <origin xyz="0 0 -0.323" rpy="0 0 ${M_PI}"/>
-        <geometry>
-          <mesh filename="package://schunk_description/meshes/lwa4d/arm_5_link.stl"/>
-        </geometry>
-        <material name="Schunk/LightGrey"/>
-      </visual>
-      <collision>
-        <origin xyz="0 0 -0.323" rpy="0 0 ${M_PI}"/>
-        <geometry>
-          <mesh filename="package://schunk_description/meshes/lwa4d/arm_5_link_collision.stl"/>
+      <!--inertial>
+        <origin xyz="0 0 0" rpy="0 0 0"/>
+        <mass value="2.313272"/>
+        <inertia ixx="0.03" ixy="0" ixz="0" iyy="0.03" iyz="0" izz="0.03" />
+      </inertial-->
+      <visual>
+        <origin xyz="0 0 -0.323" rpy="0 0 ${M_PI}" />
+        <geometry>
+          <mesh filename="package://schunk_description/meshes/lwa4d/arm_5_link.stl" />
+        </geometry>
+        <material name="Schunk/LightGrey" />
+      </visual>
+      <collision>
+        <origin xyz="0 0 -0.323" rpy="0 0 ${M_PI}" />
+        <geometry>
+          <mesh filename="package://schunk_description/meshes/lwa4d/arm_5_link.stl" />
         </geometry>
       </collision>
@@ -196,29 +194,31 @@
     <!-- joint between arm_5_link and arm_6_link -->
     <joint name="${name}_6_joint" type="revolute">
-      <origin xyz="0 0 -0.323" rpy="-${M_PI/2} 0 0"/>
+      <origin xyz="0 0 -0.323" rpy="-${M_PI/2} 0 0" />
       <parent link="${name}_5_link"/>
       <child link="${name}_6_link"/>
-      <axis xyz="0 0 1"/>
+      <axis xyz="0 0 1" />
       <calibration rising="${arm_6_ref}"/>
-      <limit effort="15" velocity="1.2566" lower="${-2.0 + safety_offset}" upper="${2.0 - safety_offset}"/>
+      <dynamics damping="5" />
+      <limit effort="15" velocity="1.2566" lower="-2.0" upper="2.0" />
+      <safety_controller k_position="20" k_velocity="25" soft_lower_limit="${-2.0 + 0.01}" soft_upper_limit="${2.0 - 0.01}" />
     </joint>
     <link name="${name}_6_link">
       <xacro:default_inertial/>
-<!--
-      <xacro:sphere_inertial radius="0.05" mass="1.9">
-        <origin xyz="0 0 0" rpy="0 0 0"/>
-      </xacro:sphere_inertial>
--->
-      <visual>
-        <origin xyz="0 0 0" rpy="0 ${M_PI} 0"/>
-        <geometry>
-          <mesh filename="package://schunk_description/meshes/lwa4d/arm_6_link.stl"/>
-        </geometry>
-        <material name="Schunk/Black"/>
-      </visual>
-      <collision>
-        <origin xyz="0 0 0" rpy="0 ${M_PI} 0"/>
-        <geometry>
-          <mesh filename="package://schunk_description/meshes/lwa4d/arm_6_link_collision.stl"/>
+      <!--inertial>
+        <origin xyz="0 0 0" rpy="0 0 0"/>
+        <mass value="2.057856"/>
+        <inertia ixx="0.01" ixy="0" ixz="0" iyy="0.01" iyz="0" izz="0.01" />
+      </inertial-->
+      <visual>
+        <origin xyz="0 0 0" rpy="0 ${M_PI} 0" />
+        <geometry>
+          <mesh filename="package://schunk_description/meshes/lwa4d/arm_6_link.stl" />
+        </geometry>
+        <material name="Schunk/Black" />
+      </visual>
+      <collision>
+        <origin xyz="0 0 0" rpy="0 ${M_PI} 0" />
+        <geometry>
+          <mesh filename="package://schunk_description/meshes/lwa4d/arm_6_link.stl" />
         </geometry>
       </collision>
@@ -226,35 +226,37 @@
     <!-- joint between arm_6_link and arm_7_link -->
     <joint name="${name}_7_joint" type="revolute">
-      <origin xyz="0 0 0" rpy="-${M_PI/2} 0 0"/>
+      <origin xyz="0 0 0" rpy="-${M_PI/2} 0 0" />
       <parent link="${name}_6_link"/>
       <child link="${name}_7_link"/>
-      <axis xyz="0 0 1"/>
+      <axis xyz="0 0 1" />
       <calibration rising="${arm_7_ref}"/>
-      <limit effort="15" velocity="1.2566" lower="${-2.0943951 + safety_offset}" upper="${2.0943951 - safety_offset}"/>
+      <dynamics damping="5" />
+      <limit effort="15" velocity="1.2566" lower="-2.967059728" upper="2.967059728" />
+      <safety_controller k_position="20" k_velocity="25" soft_lower_limit="${-2.967059728 + 0.01}" soft_upper_limit="${2.967059728 - 0.01}" />
     </joint>
     <link name="${name}_7_link">
       <xacro:default_inertial/>
-<!--
-      <xacro:cylinder_inertial radius="0.03" length="0.035" mass="0.05">
-        <origin xyz="0 0 0.06" rpy="0 0 0"/>
-      </xacro:cylinder_inertial>
--->
-      <visual>
-        <origin xyz="0 0 0.06" rpy="0 0 0"/>
-        <geometry>
-          <cylinder radius="0.03" length="0.035"/>
-        </geometry>
-        <material name="Schunk/LightGrey"/>
-      </visual>
-      <collision>
-        <origin xyz="0 0 0.06" rpy="0 0 0"/>
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
Commit message: lower vel limits: arm, gripper

File: schunk_description/urdf/lwa4d/lwa4d.urdf.xacro (robot description, xacro)
@@ -39,5 +39,5 @@
       <calibration rising="${arm_1_ref}"/>
       <dynamics damping="10" />
-      <limit effort="216" velocity="0.43633" lower="-3.1" upper="3.1"/>
+      <limit effort="216" velocity="0.3" lower="-3.1" upper="3.1"/>
       <safety_controller k_position="20" k_velocity="50" soft_lower_limit="${-3.1 + 0.01}" soft_upper_limit="${3.1 - 0.01}" />
     </joint>
@@ -72,5 +72,5 @@
       <calibration rising="${arm_2_ref}"/>
       <dynamics damping="10" />
-      <limit effort="216" velocity="0.43633" lower="-2.14" upper="2.14"/>
+      <limit effort="216" velocity="0.3" lower="-2.14" upper="2.14"/>
       <safety_controller k_position="20" k_velocity="50" soft_lower_limit="${-2.14 + 0.01}"   soft_upper_limit="${2.14 - 0.01}" />
     </joint>
@@ -104,5 +104,5 @@
       <calibration rising="${arm_3_ref}"/>
       <dynamics damping="5" />
-      <limit effort="81.5" velocity="0.4189" lower="${-M_PI}" upper="${M_PI}"/>
+      <limit effort="81.5" velocity="0.3" lower="${-M_PI}" upper="${M_PI}"/>
       <safety_controller k_position="20" k_velocity="25" soft_lower_limit="${-M_PI + 0.01}" soft_upper_limit="${M_PI - 0.01}" />
     </joint>
@@ -136,5 +136,5 @@
       <calibration rising="${arm_4_ref}"/>
       <dynamics damping="5" />
-      <limit effort="176" velocity="2.0" lower="-2.18" upper="2.18"/>
+      <limit effort="176" velocity="0.3" lower="-2.18" upper="2.18"/>
       <safety_controller k_position="20" k_velocity="25" soft_lower_limit="${-2.18 + 0.01}" soft_upper_limit="${2.18 - 0.01}" />
     </joint>
@@ -168,5 +168,5 @@
       <calibration rising="${arm_5_ref}"/>
       <dynamics damping="5" />
-      <limit effort="20.7" velocity="0.43633" lower="${-M_PI}" upper="${M_PI}" />
+      <limit effort="20.7" velocity="0.3" lower="${-M_PI}" upper="${M_PI}" />
       <safety_controller k_position="20" k_velocity="25" soft_lower_limit="${-M_PI + 0.01}" soft_upper_limit="${M_PI - 0.01}" />
     </joint>
@@ -197,8 +197,8 @@
       <parent link="${name}_5_link"/>
       <child link="${name}_6_link"/>
-      <axis xyz="0 0 1" />
+      <axis xyz="0 0 -1" />
       <calibration rising="${arm_6_ref}"/>
       <dynamics damping="5" />
-      <limit effort="15" velocity="1.2566" lower="-2.0" upper="2.0" />
+      <limit effort="15" velocity="0.3" lower="-2.0" upper="2.0" />
       <safety_controller k_position="20" k_velocity="25" soft_lower_limit="${-2.0 + 0.01}" soft_upper_limit="${2.0 - 0.01}" />
     </joint>
@@ -232,5 +232,5 @@
       <calibration rising="${arm_7_ref}"/>
       <dynamics damping="5" />
-      <limit effort="15" velocity="1.2566" lower="-2.967059728" upper="2.967059728" />
+      <limit effort="15" velocity="0.3" lower="-2.967059728" upper="2.967059728" />
       <safety_controller k_position="20" k_velocity="25" soft_lower_limit="${-2.967059728 + 0.01}" soft_upper_limit="${2.967059728 - 0.01}" />
     </joint>

File: schunk_description/urdf/pg70/pg70.transmission.xacro (robot description, xacro)
@@ -11,5 +11,5 @@
       </joint>
       <actuator name="${name}_finger_left_motor">
-        <mechanicalReduction>0.5</mechanicalReduction>
+        <mechanicalReduction>1.0</mechanicalReduction>
       </actuator>
     </transmission>
@@ -23,5 +23,5 @@
       </joint>
       <actuator name="${name}_finger_right_motor">
-        <mechanicalReduction>0.5</mechanicalReduction>
+        <mechanicalReduction>1.0</mechanicalReduction>
       </actuator>
     </transmission>

File: schunk_description/urdf/pg70/pg70.urdf.xacro (robot description, xacro)
@@ -37,5 +37,5 @@
       <parent link="${name}_gripper_link" />
       <child link="${name}_finger_left_link" />
-      <limit effort="100" lower="-0.001" upper="0.033" velocity="2.0"/>
+      <limit effort="100" lower="-0.001" upper="0.033" velocity="0.01"/>
       <calibration rising="${pg70_finger_left_ref}"/>
       <origin xyz="0 0.01 ${0.078}" rpy="0 0 0"/>
@@ -46,5 +46,5 @@
         <origin xyz="0 0 0" rpy="0 0 0"/>
         <mass value="1"/>
-        <inertia ixx="0.009" ixy="0" ixz="0" iyy="0.01" iyz="0" izz="0.01" />
+        <inertia ixx="0.009" ixy="0" ixz="0" iyy="0.01" iyz="0" izz="0.05" />
       </inertial>
       <visual>
@@ -71,5 +71,5 @@
       <parent link="${name}_gripper_link" />
       <child link="${name}_finger_right_link" />
-      <limit effort="100" lower="-0.001" upper="0.033" velocity="2.0"/>
+      <limit effort="100" lower="-0.001" upper="0.033" velocity="0.01"/>
       <calibration rising="${pg70_finger_right_ref}"/>
       <origin xyz="0 -0.009 ${0.078}" rpy="-0 0 0"/>
@@ -80,5 +80,5 @@
         <origin xyz="0 0 0" rpy="0 0 0"/>
         <mass value="1"/>
-        <inertia ixx="0.01" ixy="0" ixz="0" iyy="0.01" iyz="0" izz="0.01" />
+        <inertia ixx="0.01" ixy="0" ixz="0" iyy="0.01" iyz="0" izz="0.05" />
       </inertial>
       <visual>
