Commit message: removed inverted axis, lower arm limits

File: schunk_description/urdf/lwa4d/lwa4d.urdf.xacro (robot description, xacro)
@@ -39,5 +39,5 @@
       <calibration rising="${arm_1_ref}"/>
       <dynamics damping="10" />
-      <limit effort="216" velocity="0.3" lower="-3.1" upper="3.1"/>
+      <limit effort="216" velocity="0.2" lower="-3.1" upper="3.1"/>
       <safety_controller k_position="20" k_velocity="50" soft_lower_limit="${-3.1 + 0.01}" soft_upper_limit="${3.1 - 0.01}" />
     </joint>
@@ -72,5 +72,5 @@
       <calibration rising="${arm_2_ref}"/>
       <dynamics damping="10" />
-      <limit effort="216" velocity="0.3" lower="-2.14" upper="2.14"/>
+      <limit effort="216" velocity="0.2" lower="-2.14" upper="2.14"/>
       <safety_controller k_position="20" k_velocity="50" soft_lower_limit="${-2.14 + 0.01}"   soft_upper_limit="${2.14 - 0.01}" />
     </joint>
@@ -104,5 +104,5 @@
       <calibration rising="${arm_3_ref}"/>
       <dynamics damping="5" />
-      <limit effort="81.5" velocity="0.3" lower="${-M_PI}" upper="${M_PI}"/>
+      <limit effort="81.5" velocity="0.2" lower="${-M_PI}" upper="${M_PI}"/>
       <safety_controller k_position="20" k_velocity="25" soft_lower_limit="${-M_PI + 0.01}" soft_upper_limit="${M_PI - 0.01}" />
     </joint>
@@ -136,5 +136,5 @@
       <calibration rising="${arm_4_ref}"/>
       <dynamics damping="5" />
-      <limit effort="176" velocity="0.3" lower="-2.18" upper="2.18"/>
+      <limit effort="176" velocity="0.2" lower="-2.18" upper="2.18"/>
       <safety_controller k_position="20" k_velocity="25" soft_lower_limit="${-2.18 + 0.01}" soft_upper_limit="${2.18 - 0.01}" />
     </joint>
@@ -197,5 +197,5 @@
       <parent link="${name}_5_link"/>
       <child link="${name}_6_link"/>
-      <axis xyz="0 0 -1" />
+      <axis xyz="0 0 1" />
       <calibration rising="${arm_6_ref}"/>
       <dynamics damping="5" />

Commit message: changed finger and limits of arm

File: schunk_description/urdf/lwa4d/lwa4d.urdf.xacro (robot description, xacro)
@@ -1,4 +1,5 @@
 <?xml version="1.0"?>
 <robot xmlns:xacro="http://www.ros.org/wiki/xacro">
+  <property name="safety_offset" value="0.02"/>
   <xacro:include filename="$(find schunk_description)/urdf/lwa4d/lwa4d.gazebo.xacro" />
   <xacro:include filename="$(find schunk_description)/urdf/lwa4d/lwa4d.transmission.xacro" />
@@ -39,6 +40,5 @@
       <calibration rising="${arm_1_ref}"/>
       <dynamics damping="10" />
-      <limit effort="216" velocity="0.2" lower="-3.1" upper="3.1"/>
-      <safety_controller k_position="20" k_velocity="50" soft_lower_limit="${-3.1 + 0.01}" soft_upper_limit="${3.1 - 0.01}" />
+      <limit effort="216" velocity="0.43633" lower="${-M_PI+safety_offset}" upper="${M_PI-safety_offset}"/>
     </joint>
     <link name="${name}_1_link">
@@ -72,6 +72,5 @@
       <calibration rising="${arm_2_ref}"/>
       <dynamics damping="10" />
-      <limit effort="216" velocity="0.2" lower="-2.14" upper="2.14"/>
-      <safety_controller k_position="20" k_velocity="50" soft_lower_limit="${-2.14 + 0.01}"   soft_upper_limit="${2.14 - 0.01}" />
+      <limit effort="216" velocity="0.43633" lower="${-2.14 + safety_offset}" upper="${2.14 - safety_offset}"/>
     </joint>
     <link name="${name}_2_link">
@@ -104,6 +103,5 @@
       <calibration rising="${arm_3_ref}"/>
       <dynamics damping="5" />
-      <limit effort="81.5" velocity="0.2" lower="${-M_PI}" upper="${M_PI}"/>
-      <safety_controller k_position="20" k_velocity="25" soft_lower_limit="${-M_PI + 0.01}" soft_upper_limit="${M_PI - 0.01}" />
+      <limit effort="81.5" velocity="0.4189" lower="${-M_PI + safety_offset}" upper="${M_PI - safety_offset}"/>
     </joint>
     <link name="${name}_3_link">
@@ -136,6 +134,5 @@
       <calibration rising="${arm_4_ref}"/>
       <dynamics damping="5" />
-      <limit effort="176" velocity="0.2" lower="-2.18" upper="2.18"/>
-      <safety_controller k_position="20" k_velocity="25" soft_lower_limit="${-2.18 + 0.01}" soft_upper_limit="${2.18 - 0.01}" />
+      <limit effort="81.5" velocity="0.4189" lower="${-2.18 + safety_offset}" upper="${2.18 - safety_offset}"/>
     </joint>
     <link name="${name}_4_link">
@@ -168,6 +165,5 @@
       <calibration rising="${arm_5_ref}"/>
       <dynamics damping="5" />
-      <limit effort="20.7" velocity="0.3" lower="${-M_PI}" upper="${M_PI}" />
-      <safety_controller k_position="20" k_velocity="25" soft_lower_limit="${-M_PI + 0.01}" soft_upper_limit="${M_PI - 0.01}" />
+      <limit effort="20.7" velocity="0.43633" lower="${-M_PI + safety_offset}" upper="${M_PI - safety_offset}"/>
     </joint>
     <link name="${name}_5_link">
@@ -200,6 +196,5 @@
       <calibration rising="${arm_6_ref}"/>
       <dynamics damping="5" />
-      <limit effort="15" velocity="0.3" lower="-2.0" upper="2.0" />
-      <safety_controller k_position="20" k_velocity="25" soft_lower_limit="${-2.0 + 0.01}" soft_upper_limit="${2.0 - 0.01}" />
+      <limit effort="15" velocity="1.2566" lower="${-2.09 + safety_offset}" upper="${2.09 - safety_offset}"/>
     </joint>
     <link name="${name}_6_link">
@@ -232,6 +227,5 @@
       <calibration rising="${arm_7_ref}"/>
       <dynamics damping="5" />
-      <limit effort="15" velocity="0.3" lower="-2.967059728" upper="2.967059728" />
-      <safety_controller k_position="20" k_velocity="25" soft_lower_limit="${-2.967059728 + 0.01}" soft_upper_limit="${2.967059728 - 0.01}" />
+      <limit effort="15" velocity="1.2566" lower="${-2.96 + safety_offset}" upper="${2.96 - safety_offset}"/>
     </joint>
     <link name="${name}_7_link">
