Commit message: added finger mesh

File: schunk_description/urdf/pg70/pg70.urdf.xacro (robot description, xacro)
@@ -16,4 +16,5 @@
       </inertial>
       <visual>
+      	<origin xyz="0 0 0.0075" rpy="0 0 0"/>
         <geometry>
           <mesh filename="package://schunk_description/meshes/pg70/pg70.dae" />
@@ -24,4 +25,5 @@
       </visual>
       <collision>
+      	<origin xyz="0 0 0.0075" rpy="0 0 0"/>
         <geometry>
           <mesh filename="package://schunk_description/meshes/pg70/pg70.dae" />
@@ -37,5 +39,5 @@
       <limit effort="100" lower="-0.001" upper="0.033" velocity="2.0"/>
       <calibration rising="${pg70_finger_left_ref}"/>
-      <origin xyz="0 0.0105 ${0.0789-0.01}" rpy="0 0 0"/>
+      <origin xyz="0 0.01 ${0.078}" rpy="0 0 0"/>
       <axis xyz="0 1 0" />
     </joint>
@@ -44,17 +46,17 @@
         <origin xyz="0 0 0" rpy="0 0 0"/>
         <mass value="1"/>
-        <inertia ixx="0.01" ixy="0" ixz="0" iyy="0.01" iyz="0" izz="0.01" />
+        <inertia ixx="0.009" ixy="0" ixz="0" iyy="0.01" iyz="0" izz="0.01" />
       </inertial>
       <visual>
-        <origin xyz="0 0 0.05" rpy="0 0 0" />
+        <origin xyz="0 0 0.06" rpy="3.14159 0 0" />
         <geometry>
-          <box size="0.03 0.02 0.10"/>
+          <mesh filename="package://schunk_description/meshes/pg70/RobotGripperLongV2.stl" scale="0.001 0.001 0.001"/>
         </geometry>
-        <material name="black">
-          <color rgba="0 0 0 1"/>
+        <material name="blue">
+          <color rgba="0 0 255 1"/>
         </material>
       </visual>
       <collision>
-        <origin xyz="0 0 0.05" rpy="0 0 0" />
+        <origin xyz="0 0 0.06" rpy="0 0 0" />
         <geometry>
           <box size="0.03 0.02 0.10"/>
@@ -71,5 +73,5 @@
       <limit effort="100" lower="-0.001" upper="0.033" velocity="2.0"/>
       <calibration rising="${pg70_finger_right_ref}"/>
-      <origin xyz="0 -0.0105 ${0.0789-0.01}" rpy="-0 0 0"/>
+      <origin xyz="0 -0.009 ${0.078}" rpy="-0 0 0"/>
       <axis xyz="0 -1 0" />
     </joint>
@@ -81,14 +83,14 @@
       </inertial>
       <visual>
-        <origin xyz="0 0 0.05" rpy="0 0 0" />
+        <origin xyz="0 0 0.06" rpy="3.14159 0 3.14159" />
         <geometry>
-          <box size="0.03 0.02 0.10"/>
+          <mesh filename="package://schunk_description/meshes/pg70/RobotGripperLongV2.stl" scale="0.001 0.001 0.001"/>
         </geometry>
-        <material name="black">
-          <color rgba="0 0 0 1"/>
+        <material name="blue">
+          <color rgba="0 0 255 1"/>
         </material>
       </visual>
       <collision>
-        <origin xyz="0 0 0.05" rpy="0 0 0" />
+        <origin xyz="0 0 0.06" rpy="0 0 0" />
         <geometry>
           <box size="0.03 0.02 0.10"/>

Commit message: pg70 gripper changed

File: schunk_description/urdf/pg70/pg70.urdf.xacro (robot description, xacro)
@@ -4,10 +4,10 @@
   <xacro:include filename="$(find schunk_description)/urdf/pg70/pg70.transmission.xacro" />
   <xacro:macro name="schunk_pg70" params="parent name *origin pg70_finger_left_ref pg70_finger_right_ref">
-    <joint name="${name}_palm_joint" type="fixed" >
+    <joint name="${name}_gripper_joint" type="fixed" >
       <parent link="${parent}" />
-      <child link="${name}_palm_link" />
+      <child link="${name}_gripper_link" />
       <xacro:insert_block name="origin" />
     </joint>
-    <link name="${name}_palm_link">
+    <link name="${name}_gripper_link">
       <inertial>
         <origin xyz="0 0 0" rpy="0 0 0"/>
@@ -35,5 +35,5 @@
     </link>
     <joint name="${name}_finger_left_joint" type="prismatic" >
-      <parent link="${name}_palm_link" />
+      <parent link="${name}_gripper_link" />
       <child link="${name}_finger_left_link" />
       <limit effort="100" lower="-0.001" upper="0.033" velocity="2.0"/>
@@ -58,10 +58,10 @@
       </visual>
       <collision>
-        <origin xyz="0 0 0.06" rpy="0 0 0" />
+        <origin xyz="0 0 0.06" rpy="3.14159 0 0" />
         <geometry>
-          <box size="0.03 0.02 0.10"/>
+          <mesh filename="package://schunk_description/meshes/pg70/RobotGripperLongV2.stl" scale="0.001 0.001 0.001"/>
         </geometry>
-        <material name="black">
-          <color rgba="0 0 0 1"/>
+        <material name="blue">
+          <color rgba="0 0 255 1"/>
         </material>
       </collision>
@@ -69,5 +69,5 @@
     <joint name="${name}_finger_right_joint" type="prismatic" >
       <mimic joint="${name}_finger_left_joint" multiplier="1" offset="0"/>
-      <parent link="${name}_palm_link" />
+      <parent link="${name}_gripper_link" />
       <child link="${name}_finger_right_link" />
       <limit effort="100" lower="-0.001" upper="0.033" velocity="2.0"/>

Commit message: new finger

File: schunk_description/urdf/pg70/pg70.urdf.xacro (robot description, xacro)
@@ -49,19 +49,19 @@
       </inertial>
       <visual>
-        <origin xyz="0 0 0.06" rpy="3.14159 0 0" />
+        <origin xyz="-0.015 0.0155 0.055" rpy="3.14159 -1.57 0" />
         <geometry>
-          <mesh filename="package://schunk_description/meshes/pg70/RobotGripperLongV2.stl" scale="0.001 0.001 0.001"/>
+          <mesh filename="package://schunk_description/meshes/pg70/finger_2cm.stl" scale="0.001 0.001 0.001"/>
         </geometry>
-        <material name="blue">
-          <color rgba="0 0 255 1"/>
+        <material name="green">
+          <color rgba="0 255 0 1"/>
         </material>
       </visual>
       <collision>
-        <origin xyz="0 0 0.06" rpy="3.14159 0 0" />
+        <origin xyz="-0.015 0.0155 0.055" rpy="3.14159 -1.57 0" />
         <geometry>
-          <mesh filename="package://schunk_description/meshes/pg70/RobotGripperLongV2.stl" scale="0.001 0.001 0.001"/>
+          <mesh filename="package://schunk_description/meshes/pg70/finger_2cm.stl" scale="0.001 0.001 0.001"/>
         </geometry>
-        <material name="blue">
-          <color rgba="0 0 255 1"/>
+        <material name="green">
+          <color rgba="0 255 0 1"/>
         </material>
       </collision>
@@ -83,19 +83,19 @@
       </inertial>
       <visual>
-        <origin xyz="0 0 0.06" rpy="3.14159 0 3.14159" />
+        <origin xyz="0.015 -0.0155 0.055" rpy="3.14159 -1.57 3.14159" />
         <geometry>
-          <mesh filename="package://schunk_description/meshes/pg70/RobotGripperLongV2.stl" scale="0.001 0.001 0.001"/>
+          <mesh filename="package://schunk_description/meshes/pg70/finger_2cm.stl" scale="0.001 0.001 0.001"/>
         </geometry>
-        <material name="blue">
-          <color rgba="0 0 255 1"/>
+        <material name="red">
+          <color rgba="255 0 0 1"/>
         </material>
       </visual>
       <collision>
-        <origin xyz="0 0 0.06" rpy="0 0 0" />
+        <origin xyz="0.015 -0.0155 0.055" rpy="3.14159 -1.57 3.14159" />
         <geometry>
-          <box size="0.03 0.02 0.10"/>
+          <mesh filename="package://schunk_description/meshes/pg70/finger_2cm.stl" scale="0.001 0.001 0.001"/>
         </geometry>
-        <material name="black">
-          <color rgba="0 0 0 1"/>
+        <material name="red">
+          <color rgba="255 0 0 1"/>
         </material>
       </collision>

Commit message: dae statt stl

File: schunk_description/urdf/pg70/pg70.urdf.xacro (robot description, xacro)
@@ -51,5 +51,5 @@
         <origin xyz="-0.015 0.0155 0.055" rpy="3.14159 -1.57 0" />
         <geometry>
-          <mesh filename="package://schunk_description/meshes/pg70/finger_2cm.stl" scale="0.001 0.001 0.001"/>
+          <mesh filename="package://schunk_description/meshes/pg70/finger_2cm.dae" scale="0.001 0.001 0.001"/>
         </geometry>
         <material name="green">
@@ -60,5 +60,5 @@
         <origin xyz="-0.015 0.0155 0.055" rpy="3.14159 -1.57 0" />
         <geometry>
-          <mesh filename="package://schunk_description/meshes/pg70/finger_2cm.stl" scale="0.001 0.001 0.001"/>
+          <mesh filename="package://schunk_description/meshes/pg70/finger_2cm.dae" scale="0.001 0.001 0.001"/>
         </geometry>
         <material name="green">
@@ -85,5 +85,5 @@
         <origin xyz="0.015 -0.0155 0.055" rpy="3.14159 -1.57 3.14159" />
         <geometry>
-          <mesh filename="package://schunk_description/meshes/pg70/finger_2cm.stl" scale="0.001 0.001 0.001"/>
+          <mesh filename="package://schunk_description/meshes/pg70/finger_2cm.dae" scale="0.001 0.001 0.001"/>
         </geometry>
         <material name="red">
@@ -94,5 +94,5 @@
         <origin xyz="0.015 -0.0155 0.055" rpy="3.14159 -1.57 3.14159" />
         <geometry>
-          <mesh filename="package://schunk_description/meshes/pg70/finger_2cm.stl" scale="0.001 0.001 0.001"/>
+          <mesh filename="package://schunk_description/meshes/pg70/finger_2cm.dae" scale="0.001 0.001 0.001"/>
         </geometry>
         <material name="red">
